File: IGBT DRIVER.sch (KiCad schematic (older format))
At the start: 42 parts, among them J1 Conn_02x05_Odd_Even, J2 Screw_Terminal_01x01, J3 Screw_Terminal_01x01, J4 Conn_01x02, J5 Conn_01x02, U1 miw06-24s24, U11 L7833s(D2pack), U2 miw06-24s24

Commit message: ..
Parts:
- G1: symbol koalaLogo:LOGO -> IGBT-DRIVER-rescue:LOGO-koalaLogo
- U1, U2: symbol GateDriver:miw06-24s24 -> IGBT-DRIVER-rescue:miw06-24s24-GateDriver
Changed lines of the file:
@@
 $EndComp
 $Comp
-L GateDriver:miw06-24s24 U2
+L IGBT-DRIVER-rescue:miw06-24s24-GateDriver U2
 U 1 1 619584B7
 P 2605 1025
@@
 $EndComp
 $Comp
-L GateDriver:miw06-24s24 U1
+L IGBT-DRIVER-rescue:miw06-24s24-GateDriver U1
 U 1 1 61959EFB
 P 2290 3585
@@
 	3160 4175 3335 4175
 $Comp
-L koalaLogo:LOGO G1
+L IGBT-DRIVER-rescue:LOGO-koalaLogo G1
 U 1 1 619E54B4
 P 1360 5435
